File: hwd/hwd_reactive/output.kicad_sch (KiCad schematic)
At the start: 27 parts

Commit message: added code for testing
Parts:
- removed R? (x23): R, symbol Device:R
- removed U? (x3): 74HC137, symbol 74xx:74HC137
- added C?: 100nF, symbol Device:C
- added R? (x23): R150, symbol Device:R
- added R? (x2): R270, symbol Device:R
- added U? (x3): 74HC595, symbol 74xx:74HC595
- added U?: MOC3063M, symbol Relay_SolidState:MOC3063M
- R8: renamed from R?; value R -> R270
Connections:
- net at R8.1: now also U?.15 (QA)
- net at R8.2: now also U?.1
- new net: R?.1, U?.15 (QA) (x2)
- new net: R?.1, U?.4 (QE) (x3)
- new net: R?.1, U?.5 (QF) (x3)
- new net: R?.1, U?.1 (QB) (x3)
- new net: U?.14 (SER), U?.9 (QH') (x2)
- new net: R?.1, U?.2 (QC) (x3)
- new net: R?.1, U?.3 (QD) (x3)
- new net: R?.1, U?.6 (QG) (x3)
- new net: R?.1, U?.7 (QH) (x3)
- new net +5V: U?.10 (~{SRCLR}), U?.16 (VCC)
- new net GND: C?.2, U?.8 (GND), U?.8 (GND), U?.8 (GND)
- new net LATCH: U?.12 (RCLK), U?.12 (RCLK), U?.12 (RCLK)
- new net SIPO_DATA: U?.14 (SER)
- new net SIPO_SCK: U?.11 (SRCLK), U?.11 (SRCLK), U?.11 (SRCLK)
- new net VCC: C?.1, U?.10 (~{SRCLR}), U?.10 (~{SRCLR}), U?.16 (VCC), U?.16 (VCC)
Other:
- moved on the sheet: R8
