File: hwd/hwd_reactive/power.kicad_sch (KiCad schematic)
At the start: 11 parts

Commit message: added code for testing
Parts:
- C10: renamed from C?; value C_Polarized -> 100uF
- C8: renamed from C?; value C_Polarized -> 10uF
- C9: renamed from C?; value C_Polarized -> 820uF
- L1: renamed from L?; value L -> 1.2uH
- L2: renamed from L?; value L -> 4.7uH
- R7: renamed from R?; value R -> R12
- gave numbers to parts that had none: 5
Changed lines of the file:
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@@
 		(dnp no)
 		(fields_autoplaced yes)
-		(property "Reference" "C?"
+		(property "Reference" "C10"
 			(at 144.78 57.5309 0)
 			(effects
@@
 			)
 		)
-		(property "Value" "C_Polarized"
+		(property "Value" "100uF"
 			(at 144.78 60.0709 0)
 			(effects
@@
 			(project "hwd_reactive"
 				(path "/e1902c4a-c8d3-47e8-8764-2534e0bb1d7a/2d2419ef-eca4-4152-a4ca-42af1a3cafa1"
-					(reference "C?")
+					(reference "C10")
 					(unit 1)
 				)
@@
 		(dnp no)
 		(fields_autoplaced yes)
-		(property "Reference" "F?"
+		(property "Reference" "F1"
 			(at 36.195 46.99 0)
 			(effects
@@
 			(project ""
 				(path "/e1902c4a-c8d3-47e8-8764-2534e0bb1d7a/2d2419ef-eca4-4152-a4ca-42af1a3cafa1"
-					(reference "F?")
+					(reference "F1")
 					(unit 1)
 				)
@@
 		(dnp no)
 		(fields_autoplaced yes)
-		(property "Reference" "C?"
+		(property "Reference" "C8"
 			(at 74.93 57.5309 0)
 			(effects
@@
 			)
 		)
-		(property "Value" "C_Polarized"
+		(property "Value" "10uF"
 			(at 74.93 60.0709 0)
 			(effects
@@
 			(project ""
 				(path "/e1902c4a-c8d3-47e8-8764-2534e0bb1d7a/2d2419ef-eca4-4152-a4ca-42af1a3cafa1"
-					(reference "C?")
+					(reference "C8")
 					(unit 1)
 				)
@@
 		(dnp no)
 		(fields_autoplaced yes)
-		(property "Reference" "D?"
+		(property "Reference" "D4"
 			(at 160.655 58.4199 90)
 			(effects
@@
 			(project ""
 				(path "/e1902c4a-c8d3-47e8-8764-2534e0bb1d7a/2d2419ef-eca4-4152-a4ca-42af1a3cafa1"
-					(reference "D?")
+					(reference "D4")
 					(unit 1)
 				)
@@
 		(dnp no)
 		(fields_autoplaced yes)
-		(property "Reference" "L?"
+		(property "Reference" "L2"
 			(at 128.905 46.99 90)
 			(effects
@@
 			)
 		)
-		(property "Value" "L"
+		(property "Value" "4.7uH"
 			(at 128.905 49.53 90)
 			(effects
@@
 			(project "hwd_reactive"
 				(path "/e1902c4a-c8d3-47e8-8764-2534e0bb1d7a/2d2419ef-eca4-4152-a4ca-42af1a3cafa1"
-					(reference "L?")
+					(reference "L2")
 					(unit 1)
 				)
@@
 		(dnp no)
 		(fields_autoplaced yes)
-		(property "Reference" "R?"
+		(property "Reference" "R7"
 			(at 50.165 45.72 90)
 			(effects
@@
 			)
 		)
-		(property "Value" "R"
+		(property "Value" "R12"
 			(at 50.165 48.26 90)
 			(effects
@@
 			(project ""
 				(path "/e1902c4a-c8d3-47e8-8764-2534e0bb1d7a/2d2419ef-eca4-4152-a4ca-42af1a3cafa1"
-					(reference "R?")
+					(reference "R7")
 					(unit 1)
 				)
@@
 		(dnp no)
 		(fields_autoplaced yes)
-		(property "Reference" "RV?"
+		(property "Reference" "RV1"
 			(at 45.72 57.9782 0)
 			(effects
@@
 			(project ""
 				(path "/e1902c4a-c8d3-47e8-8764-2534e0bb1d7a/2d2419ef-eca4-4152-a4ca-42af1a3cafa1"
-					(reference "RV?")
+					(reference "RV1")
 					(unit 1)
 				)
@@
 		(dnp no)
 		(fields_autoplaced yes)
-		(property "Reference" "C?"
+		(property "Reference" "C7"
 			(at 60.96 57.7849 0)
 			(effects
@@
 			(project ""
 				(path "/e1902c4a-c8d3-47e8-8764-2534e0bb1d7a/2d2419ef-eca4-4152-a4ca-42af1a3cafa1"
-					(reference "C?")
+					(reference "C7")
 					(unit 1)
 				)
@@
 		(dnp no)
 		(fields_autoplaced yes)
-		(property "Reference" "L?"
+		(property "Reference" "L1"
 			(at 64.135 46.99 90)
 			(effects
@@
 			)
 		)
-		(property "Value" "L"
+		(property "Value" "1.2uH"
 			(at 64.135 49.53 90)
 			(effects
@@
 			(project ""
 				(path "/e1902c4a-c8d3-47e8-8764-2534e0bb1d7a/2d2419ef-eca4-4152-a4ca-42af1a3cafa1"
-					(reference "L?")
+					(reference "L1")
 					(unit 1)
 				)
@@
 		(dnp no)
 		(fields_autoplaced yes)
-		(property "Reference" "C?"
-			(at 125.095 56.2609 0)
-			(effects
-				(font
-					(size 1.27 1.27)
-				)
-				(justify left)
-			)
-		)
-		(property "Value" "C_Polarized"
-			(at 125.095 58.8009 0)
+		(property "Reference" "C9"
+			(at 124.46 56.2609 0)
+			(effects
+				(font
+					(size 1.27 1.27)
+				)
+				(justify left)
+			)
+		)
+		(property "Value" "820uF"
+			(at 124.46 58.8009 0)
 			(effects
 				(font
@@
 			(project "hwd_reactive"
 				(path "/e1902c4a-c8d3-47e8-8764-2534e0bb1d7a/2d2419ef-eca4-4152-a4ca-42af1a3cafa1"
-					(reference "C?")
+					(reference "C9")
 					(unit 1)
 				)
@@
 		(dnp no)
 		(fields_autoplaced yes)
-		(property "Reference" "U?"
+		(property "Reference" "U1"
 			(at 98.425 45.085 0)
 			(effects
@@
 			(project ""
 				(path "/e1902c4a-c8d3-47e8-8764-2534e0bb1d7a/2d2419ef-eca4-4152-a4ca-42af1a3cafa1"
-					(reference "U?")
-					(unit 1)
-				)
+					(reference "U1")
+					(unit 1)
+				)
